Commit message: Added mapping

File: description/lidar.xacro (robot description, xacro)
@@ -38,5 +38,5 @@
                 </scan>
                 <range>
-                    <min>0.3</min>
+                    <min>0.1</min>
                     <max>8</max>
                 </range>

File: description/robot.urdf.xacro (robot description, xacro)
@@ -2,8 +2,8 @@
 <robot xmlns:xacro="http://www.ros.org/wiki/xacro"  name="robot">
     <xacro:include filename="robot_core.xacro"/>
-    <!-- <xacro:include filename="gazebo_control.xacro"/> -->
-    <xacro:include filename="ros2_control.xacro"/>
+    <xacro:include filename="gazebo_control.xacro"/>
+    <!-- <xacro:include filename="ros2_control.xacro"/> -->
     <xacro:include filename="lidar.xacro"/>
-    <!-- <xacro:include filename="camera.xacro"/> -->
-    <xacro:include filename="depth_camera.xacro"/>
+    <xacro:include filename="camera.xacro"/>
+    <!-- <xacro:include filename="depth_camera.xacro"/> -->
 </robot>

File: description/robot_core.xacro (robot description, xacro)
@@ -26,9 +26,17 @@
 	<link name="base_link">
 	</link>
+	<!-- BASE_FOOTPRINT LINK -->
+	<joint name="base_footprint_joint" type="fixed">
+		<parent link="chassis"/>
+		<child link="base_footprint"/>
+		<origin xyz="0 0 0" rpy="0 0 0"/>
+	</joint>
+	<link name="base_footprint">
+	</link>
 	<!-- CHASSIS LINK -->
 	<joint name="chassis_joint" type="fixed">
 		<parent link="base_link"/>
 		<child link="chassis"/>
-		<origin xyz="0.3 0 0"/>
+		<origin xyz="0 0 0"/>
 	</joint>
 	<link name="chassis">
