Commit message: Robot driving

File: description/robot.urdf.xacro (robot description, xacro)
@@ -2,3 +2,4 @@
 <robot xmlns:xacro="http://www.ros.org/wiki/xacro"  name="robot">
     <xacro:include filename="robot_core.xacro"/>
+    <xacro:include filename="gazebo_control.xacro"/>
 </robot>

File: description/robot_core.xacro (robot description, xacro)
@@ -45,4 +45,7 @@
 		</xacro:inertial_box>
 	</link>
+	<gazebo reference="chassis">
+		<material>Gazebo/Red</material>
+	</gazebo>
 	<!-- LEFT WHEEL LINK -->
 	<joint name="left_wheel_joint" type="continuous">
@@ -69,4 +72,7 @@
 		</xacro:inertial_cylinder>
 	</link>
+	<gazebo reference="left_wheel">
+		<material>Gazebo/Blue</material>
+	</gazebo>
 	<!-- RIGHT WHEEL LINK -->
 	<joint name="right_wheel_joint" type="continuous">
@@ -93,4 +99,7 @@
 		</xacro:inertial_cylinder>
 	</link>
+	<gazebo reference="right_wheel">
+		<material>Gazebo/Blue</material>
+	</gazebo>
 	<!-- CASTER WHEEL LINK -->
 	<joint name="caster_wheel_joint" type="fixed">
@@ -116,3 +125,8 @@
 		</xacro:inertial_sphere>
 	</link>
+	<gazebo reference="caster_wheel">
+		<material>Gazebo/Black</material>
+		<mu1 value="0.001"/>
+		<mu2 value="0.001"/>
+	</gazebo>
 </robot>

Commit message: Camera was added

File: description/robot.urdf.xacro (robot description, xacro)
@@ -3,3 +3,5 @@
     <xacro:include filename="robot_core.xacro"/>
     <xacro:include filename="gazebo_control.xacro"/>
+    <xacro:include filename="lidar.xacro"/>
+    <xacro:include filename="camera.xacro"/>
 </robot>

File: description/robot_core.xacro (robot description, xacro)
@@ -4,4 +4,7 @@
 	<material name="white">
    		<color rgba="1 1 1 1"/>
+  	</material>
+  	<material name="orange">
+   		<color rgba="1 0.3 0.1 1"/>
   	</material>
 	<material name="red">
@@ -16,4 +19,7 @@
 	<material name="black">
    		<color rgba="0 0 0 1"/>
+  	</material>
+  	<material name="grey">
+   		<color rgba="0.5 0.5 0.5 1"/>
   	</material>
 	<!-- BASE LINK -->
@@ -32,5 +38,5 @@
 				<box size="0.3 0.28 0.08"/>
 			</geometry>
-			<material name="red"/>
+			<material name="white"/>
 		</visual>
 		<collision>
@@ -39,5 +45,5 @@
 				<box size="0.3 0.28 0.08"/>
 			</geometry>
-			<material name="red"/>
+			<material name="white"/>
 		</collision>
 		<xacro:inertial_box mass="1.5" x="0.3" y="0.28" z="0.08">
@@ -46,5 +52,5 @@
 	</link>
 	<gazebo reference="chassis">
-		<material>Gazebo/Red</material>
+		<material>Gazebo/White</material>
 	</gazebo>
 	<!-- LEFT WHEEL LINK -->

Commit message: Fix odometry

File: description/robot.urdf.xacro (robot description, xacro)
@@ -2,6 +2,6 @@
 <robot xmlns:xacro="http://www.ros.org/wiki/xacro"  name="robot">
     <xacro:include filename="robot_core.xacro"/>
-    <xacro:include filename="gazebo_control.xacro"/>
-    <!-- <xacro:include filename="ros2_control.xacro"/> -->
+    <!-- <xacro:include filename="gazebo_control.xacro"/> -->
+    <xacro:include filename="ros2_control.xacro"/>   <!-- Uncommit for ros2_control -->
     <xacro:include filename="lidar.xacro"/>
     <xacro:include filename="camera.xacro"/>

File: description/robot_core.xacro (robot description, xacro)
@@ -28,5 +28,5 @@
 	<!-- BASE_FOOTPRINT LINK -->
 	<joint name="base_footprint_joint" type="fixed">
-		<parent link="chassis"/>
+		<parent link="base_link"/>
 		<child link="base_footprint"/>
 		<origin xyz="0 0 0" rpy="0 0 0"/>
@@ -38,5 +38,5 @@
 		<parent link="base_link"/>
 		<child link="chassis"/>
-		<origin xyz="0 0 0"/>
+		<origin xyz="-0.09 0 0"/>
 	</joint>
 	<link name="chassis">

Commit message: Add 3 sensors

File: description/robot.urdf.xacro (robot description, xacro)
@@ -5,6 +5,7 @@
     <!-- <xacro:include filename="ros2_control.xacro"/> -->   <!-- Uncommit for ros2_control -->
     <!-- <xacro:include filename="lidar.xacro"/> -->
-    <xacro:include filename="ultrasonic.xacro"/>
-    <xacro:include filename="camera.xacro"/>
+    <xacro:include filename="ultrasonic_central.xacro"/>
+    <xacro:include filename="ultrasonic_left.xacro"/>
+    <!-- <xacro:include filename="camera.xacro"/> -->
     <!-- <xacro:include filename="depth_camera.xacro"/> -->
 </robot>

File: description/ultrasonic_central.xacro (robot description, xacro)
@@ -1,13 +1,14 @@
 <?xml version="1.0"?>
 <robot xmlns:xacro="http://www.ros.org/wiki/xacro">
-	<joint name="ultrasonic_joint" type="fixed">
+	<!-- CENTRAL ULTRASONIC SENSOR-->
+	<joint name="central_ultrasonic_joint" type="fixed">
 		<parent link="chassis"/>
-		<child link="ultrasonic_frame"/>
-		<origin xyz="0.1 0 0.1" rpy="0 0 0"/>
+		<child link="central_ultrasonic_frame"/>
+		<origin xyz="0.14 0 0.09" rpy="0 0 0"/>
 	</joint>
-	<link name="ultrasonic_frame">
+	<link name="central_ultrasonic_frame">
 		<visual>
 			<geometry>
-				<cylinder radius="0.03" length="0.04"/>
+				<box size="0.015 0.045 0.02 "/>
 			</geometry>
 			<material name="red"/>
@@ -15,13 +16,13 @@
 		<collision>
 			<geometry>
-				<cylinder radius="0.03" length="0.04"/>
+				<box size="0.015 0.045 0.02 "/>
 			</geometry>
 			<material name="red"/>
 		</collision>
-		<xacro:inertial_cylinder mass="0.1" radius="0.03" length="0.04">
-			<origin xyz="0 0 0" rpy="0 0 0"/>
-		</xacro:inertial_cylinder>
+		<xacro:inertial_box mass="0.05" x="0.015" y="0.045" z="0.02">
+			<origin xyz="0 0 0.01" rpy="0 0 0"/>
+		</xacro:inertial_box>
 	</link>
-	<gazebo reference="ultrasonic_frame">
+	<gazebo reference="central_ultrasonic_frame">
 		<material>Gazebo/Red</material>
         <sensor name="ultrasonic" type="ray">
@@ -45,6 +46,6 @@
                 </scan>
                 <range>
-                    <min>0.1</min>
-                    <max>0.5</max>
+                    <min>0.008</min>
+                    <max>1.3</max>
                     <resolution>0.01</resolution>
                 </range>
@@ -55,11 +56,11 @@
       			</noise>
             </ray>
-            <plugin name="ultrasonic_sensor_1" filename="libgazebo_ros_ray_sensor.so">
+            <plugin name="ultrasonic_sensor_central" filename="libgazebo_ros_ray_sensor.so">
                 <ros>
-                    <argument>~/out:=ultrasonic_sensor_1</argument>
+                    <argument>~/out:=ultrasonic_sensor_central</argument>
                 </ros>
                 <output_type>sensor_msgs/Range</output_type>
                 <radiation_type>ultrasound</radiation_type>
-                <frame_name>ultrasonic_frame</frame_name>
+                <frame_name>central_ultrasonic_frame</frame_name>
             </plugin>
         </sensor>

Commit message: Ultrasonic sensors work

File: description/robot.urdf.xacro (robot description, xacro)
@@ -6,4 +6,6 @@
     <!-- <xacro:include filename="lidar.xacro"/> -->
     <xacro:include filename="ultrasonic_central.xacro"/>
+    <xacro:include filename="ultrasonic_left.xacro"/>
+    <xacro:include filename="ultrasonic_right.xacro"/>
     <!-- <xacro:include filename="camera.xacro"/> -->
     <!-- <xacro:include filename="depth_camera.xacro"/> -->

File: description/ultrasonic_central.xacro (robot description, xacro)
@@ -26,5 +26,5 @@
 	<gazebo reference="central_ultrasonic_frame">
 		<material>Gazebo/Red</material>
-        <sensor name="ultrasonic" type="ray">
+        <sensor name="ultrasonic_central" type="ray">
             <pose> 0 0 0 0 0 0 </pose>
             <visualize>true</visualize>

File: description/ultrasonic_left.xacro (robot description, xacro)
@@ -26,5 +26,5 @@
 	<gazebo reference="left_ultrasonic_frame">
 		<material>Gazebo/Red</material>
-        <sensor name="ultrasonic" type="ray">
+        <sensor name="ultrasonic_left" type="ray">
             <pose> 0 0 0 0 0 0 </pose>
             <visualize>true</visualize>
@@ -66,68 +66,3 @@
         </sensor>
     </gazebo>
-    <!-- RIGHT ULTRASONIC
-	<joint name="right_ultrasonic_joint" type="fixed">
-		<parent link="chassis"/>
-		<child link="ultrasonic_frame"/>
-		<origin xyz="0.1 0 0.1" rpy="0 0 0"/>
-	</joint>
-	<link name="right_ultrasonic_frame">
-		<visual>
-			<geometry>
-				<cylinder radius="0.03" length="0.04"/>
-			</geometry>
-			<material name="red"/>
-		</visual>
-		<collision>
-			<geometry>
-				<cylinder radius="0.03" length="0.04"/>
-			</geometry>
-			<material name="red"/>
-		</collision>
-		<xacro:inertial_cylinder mass="0.1" radius="0.03" length="0.04">
-			<origin xyz="0 0 0" rpy="0 0 0"/>
-		</xacro:inertial_cylinder>
-	</link>
-	<gazebo reference="right_ultrasonic_frame">
-		<material>Gazebo/Red</material>
-        <sensor name="ultrasonic" type="ray">
-            <pose> 0 0 0 0 0 0 </pose>
-            <visualize>true</visualize>
-            <update_rate>5</update_rate>
-            <ray>
-                <scan>
-                    <horizontal>
-                        <samples>5</samples>
-                        <resolution>1.000000</resolution>
-                        <min_angle>-0.26</min_angle>
-                        <max_angle>0.26</max_angle>
-                    </horizontal>
-                    <vertical>
-          				<samples>5</samples>
-          				<resolution>1.000000</resolution>
-          				<min_angle>-0.01</min_angle>
-          				<max_angle>0.01</max_angle>
-        			</vertical>
-                </scan>
-                <range>
-                    <min>0.1</min>
-                    <max>0.5</max>
-                    <resolution>0.01</resolution>
-                </range>
-                <noise>
-        			<type>gaussian</type>
-        			<mean>0.0</mean>
-        			<stddev>0.01</stddev>
-      			</noise>
-            </ray>
-            <plugin name="ultrasonic_sensor_1" filename="libgazebo_ros_ray_sensor.so">
-                <ros>
-                    <argument>~/out:=ultrasonic_sensor_right</argument>
-                </ros>
-                <output_type>sensor_msgs/Range</output_type>
-                <radiation_type>ultrasound</radiation_type>
-                <frame_name>right_ultrasonic_frame</frame_name>
-            </plugin>
-        </sensor>
-    </gazebo> -->
 </robot>

File: description/ultrasonic_right.xacro (robot description, xacro)
@@ -1,11 +1,11 @@
 <?xml version="1.0"?>
 <robot xmlns:xacro="http://www.ros.org/wiki/xacro">
-	<!-- LEFT ULTRASONIC -->
-	<joint name="left_ultrasonic_joint" type="fixed">
+	<!-- RIGHT ULTRASONIC -->
+	<joint name="right_ultrasonic_joint" type="fixed">
 		<parent link="chassis"/>
-		<child link="left_ultrasonic_frame"/>
-		<origin xyz="0.1239 0.0389 0.09" rpy="0 0 ${pi/2}"/>
+		<child link="right_ultrasonic_frame"/>
+		<origin xyz="0.1239 -0.0389 0.09" rpy="0 0 -${pi/4}"/>
 	</joint>
-	<link name="left_ultrasonic_frame">
+	<link name="right_ultrasonic_frame">
 		<visual>
 			<geometry>
@@ -24,7 +24,7 @@
 		</xacro:inertial_box>
 	</link>
-	<gazebo reference="left_ultrasonic_frame">
+	<gazebo reference="right_ultrasonic_frame">
 		<material>Gazebo/Red</material>
-        <sensor name="ultrasonic" type="ray">
+        <sensor name="ultrasonic_right" type="ray">
             <pose> 0 0 0 0 0 0 </pose>
             <visualize>true</visualize>
@@ -56,70 +56,5 @@
       			</noise>
             </ray>
-            <plugin name="ultrasonic_sensor_2" filename="libgazebo_ros_ray_sensor.so">
-                <ros>
-                    <argument>~/out:=ultrasonic_sensor_2</argument>
-                </ros>
-                <output_type>sensor_msgs/Range</output_type>
-                <radiation_type>ultrasound</radiation_type>
-                <frame_name>left_ultrasonic_frame</frame_name>
-            </plugin>
-        </sensor>
-    </gazebo>
-    <!-- RIGHT ULTRASONIC
-	<joint name="right_ultrasonic_joint" type="fixed">
-		<parent link="chassis"/>
-		<child link="ultrasonic_frame"/>
-		<origin xyz="0.1 0 0.1" rpy="0 0 0"/>
-	</joint>
-	<link name="right_ultrasonic_frame">
-		<visual>
-			<geometry>
-				<cylinder radius="0.03" length="0.04"/>
-			</geometry>
-			<material name="red"/>
-		</visual>
-		<collision>
-			<geometry>
-				<cylinder radius="0.03" length="0.04"/>
-			</geometry>
-			<material name="red"/>
-		</collision>
-		<xacro:inertial_cylinder mass="0.1" radius="0.03" length="0.04">
-			<origin xyz="0 0 0" rpy="0 0 0"/>
-		</xacro:inertial_cylinder>
-	</link>
-	<gazebo reference="right_ultrasonic_frame">
-		<material>Gazebo/Red</material>
-        <sensor name="ultrasonic" type="ray">
-            <pose> 0 0 0 0 0 0 </pose>
-            <visualize>true</visualize>
-            <update_rate>5</update_rate>
-            <ray>
-                <scan>
-                    <horizontal>
-                        <samples>5</samples>
-                        <resolution>1.000000</resolution>
-                        <min_angle>-0.26</min_angle>
-                        <max_angle>0.26</max_angle>
-                    </horizontal>
-                    <vertical>
-          				<samples>5</samples>
-          				<resolution>1.000000</resolution>
-          				<min_angle>-0.01</min_angle>
-          				<max_angle>0.01</max_angle>
-        			</vertical>
-                </scan>
-                <range>
-                    <min>0.1</min>
-                    <max>0.5</max>
-                    <resolution>0.01</resolution>
-                </range>
-                <noise>
-        			<type>gaussian</type>
-        			<mean>0.0</mean>
-        			<stddev>0.01</stddev>
-      			</noise>
-            </ray>
-            <plugin name="ultrasonic_sensor_1" filename="libgazebo_ros_ray_sensor.so">
+            <plugin name="ultrasonic_sensor_right" filename="libgazebo_ros_ray_sensor.so">
                 <ros>
                     <argument>~/out:=ultrasonic_sensor_right</argument>
@@ -130,4 +65,4 @@
             </plugin>
         </sensor>
-    </gazebo> -->
+    </gazebo>
 </robot>
