Commit message: Update for ROS Jazzy and Gazebo Harmonic

File: description/camera.xacro (robot description, xacro)
@@ -29,4 +29,5 @@
             <update_rate>10</update_rate>
 			<camera>
+				<camera_info_topic>camera/camera_info</camera_info_topic>
                 <horizontal_fov>1.089</horizontal_fov>
                 <image>
@@ -40,7 +41,6 @@
                 </clip>
             </camera>
-            <plugin name="camera_controller" filename="libgazebo_ros_camera.so">
-                <frame_name>camera_optical_link</frame_name>
-            </plugin>
+            <topic>camera/image_raw</topic>
+            <gz_frame_id>camera_optical_link</gz_frame_id>
         </sensor>
     </gazebo>

File: description/gazebo_control.xacro (robot description, xacro)
@@ -2,20 +2,31 @@
 <robot xmlns:xacro="http://www.ros.org/wiki/xacro">
     <gazebo>
-    	<plugin name="diff_drive" filename="libgazebo_ros_diff_drive.so">
-    		<!-- Wheel Information -->
+		<plugin name="gz::sim::systems::DiffDrive" filename="gz-sim-diff-drive-system">
+			<!-- Wheel Information -->
     		<left_joint>left_wheel_joint</left_joint>
     		<right_joint>right_wheel_joint</right_joint>
     		<wheel_separation>0.31</wheel_separation>
-    		<wheel_diameter>0.08</wheel_diameter>
+			<wheel_radius>0.04</wheel_radius>
+            <!-- 0.04 -->
     		<!-- Limits -->
-    		<max_wheel_torque>200</max_wheel_torque>
-    		<max_wheel_acceleration>10.0</max_wheel_acceleration>
+    		<!-- <max_wheel_torque>200</max_wheel_torque> -->
+            <!-- <max_linear_acceleration>1.0</max_linear_acceleration> -->
+			<!-- Input -->
+            <topic>cmd_vel</topic>
     		<!-- Output -->
-    		<odometry_frame>odom</odometry_frame>
-    		<robot_base_frame>base_link</robot_base_frame>
-    		<publish_odom>true</publish_odom>
-    		<publish_odom_tf>true</publish_odom_tf>
-    		<publish_wheel_tf>true</publish_wheel_tf>
-    	</plugin>
+    		<frame_id>odom</frame_id>
+            <child_frame_id>base_link</child_frame_id>
+            <odom_topic>odom</odom_topic>
+            <odom_publisher_frequency>50</odom_publisher_frequency>
+            <tf_topic>/tf</tf_topic>
+            <update_rate>100</update_rate>
+            <odometry_source>0</odometry_source>
+        </plugin>
+		<plugin filename="gz-sim-joint-state-publisher-system"
+            name="gz::sim::systems::JointStatePublisher">
+            <topic>joint_states</topic>
+            <joint_name>left_wheel_joint</joint_name>
+            <joint_name>right_wheel_joint</joint_name>
+        </plugin>
     </gazebo>
 </robot>

File: description/lidar.xacro (robot description, xacro)
@@ -25,9 +25,9 @@
 	<gazebo reference="lidar_frame">
 		<material>Gazebo/Red</material>
-        <sensor name="lidar" type="ray">
-            <pose> 0 0 0 0 0 0 </pose>
+        <sensor name="laser" type="gpu_lidar">
+            <!-- <ignition_frame_id>custom_name_here</ignition_frame_id>             <pose> 0 0 0 0 0 0 </pose> -->
             <visualize>false</visualize>
             <update_rate>10</update_rate>
-            <ray>
+            <lidar>
                 <scan>
                     <horizontal>
@@ -41,12 +41,7 @@
                     <max>8</max>
                 </range>
-            </ray>
-            <plugin name="laser_controller" filename="libgazebo_ros_ray_sensor.so">
-                <ros>
-                    <argument>~/out:=scan</argument>
-                </ros>
-                <output_type>sensor_msgs/LaserScan</output_type>
-                <frame_name>lidar_frame</frame_name>
-            </plugin>
+            </lidar>
+            <topic>scan</topic>
+            <gz_frame_id>lidar_frame</gz_frame_id>
         </sensor>
     </gazebo>

File: description/robot.urdf.xacro (robot description, xacro)
@@ -3,11 +3,8 @@
     <xacro:include filename="robot_core.xacro"/>
     <xacro:include filename="gazebo_control.xacro"/>
-    <!-- <xacro:include filename="ros2_control.xacro"/> -->   <!-- Uncommit for ros2_control -->
-    <!-- <xacro:include filename="lidar.xacro"/> -->
-    <xacro:include filename="ultrasonics.xacro"/>
-    <!-- <xacro:include filename="ultrasonic_central.xacro"/>
-    <xacro:include filename="ultrasonic_left.xacro"/>
-    <xacro:include filename="ultrasonic_right.xacro"/> -->
-    <!-- <xacro:include filename="camera.xacro"/> -->
+    <!-- <xacro:include filename="ros2_control.xacro"/>   Uncommit for ros2_control -->
+    <xacro:include filename="lidar.xacro"/>
+    <!-- <xacro:include filename="tof_sensors.xacro"/> -->
+    <xacro:include filename="camera.xacro"/>
     <!-- <xacro:include filename="depth_camera.xacro"/> -->
 </robot>

File: description/robot_core.xacro (robot description, xacro)
@@ -38,5 +38,5 @@
 		<parent link="base_link"/>
 		<child link="chassis"/>
-		<origin xyz="-0.09 0 0"/>
+		<origin xyz="0 0 0" rpy="0 0 0"/>
 	</joint>
 	<link name="chassis">
@@ -55,5 +55,5 @@
 			<material name="white"/>
 		</collision>
-		<xacro:inertial_box mass="1.5" x="0.3" y="0.28" z="0.08">
+		<xacro:inertial_box mass="2" x="0.3" y="0.28" z="0.08">
 			<origin xyz="0 0 0.04" rpy="0 0 0"/>
 		</xacro:inertial_box>
@@ -66,5 +66,5 @@
 		<parent link="chassis"/>
 		<child link="left_wheel"/>
-		<origin xyz="0.09 0.155 0" rpy="-${pi/2} 0 0"/>
+		<origin xyz="0 0.155 0" rpy="-${pi/2} 0 0"/>
 		<axis xyz="0 0 1"/>
 	</joint>
@@ -82,5 +82,5 @@
 			<material name="blue"/>
 		</collision>
-		<xacro:inertial_cylinder mass="0.1" radius="0.04" length="0.03">
+		<xacro:inertial_cylinder mass="0.5" radius="0.04" length="0.03">
 			<origin xyz="0 0 0" rpy="0 0 0"/>
 		</xacro:inertial_cylinder>
@@ -93,5 +93,5 @@
 		<parent link="chassis"/>
 		<child link="right_wheel"/>
-		<origin xyz="0.09 -0.155 0" rpy="${pi/2} 0 0"/>
+		<origin xyz="0 -0.155 0" rpy="${pi/2} 0 0"/>
 		<axis xyz="0 0 -1"/>
 	</joint>
@@ -109,5 +109,5 @@
 			<material name="blue"/>
 		</collision>
-		<xacro:inertial_cylinder mass="0.1" radius="0.04" length="0.03">
+		<xacro:inertial_cylinder mass="0.5" radius="0.04" length="0.03">
 			<origin xyz="0 0 0" rpy="0 0 0"/>
 		</xacro:inertial_cylinder>
@@ -116,11 +116,11 @@
 		<material>Gazebo/Blue</material>
 	</gazebo>
-	<!-- CASTER WHEEL LINK -->
-	<joint name="caster_wheel_joint" type="fixed">
+	<!-- CASTER WHEEL LINK BACK -->
+	<joint name="caster_wheel_joint_back" type="fixed">
 		<parent link="chassis"/>
-		<child link="caster_wheel"/>
+		<child link="caster_wheel_back"/>
 		<origin xyz="-0.1 0 0"/>
 	</joint>
-	<link name="caster_wheel">
+	<link name="caster_wheel_back">
 		<visual>
 			<geometry>
@@ -139,5 +139,33 @@
 		</xacro:inertial_sphere>
 	</link>
-	<gazebo reference="caster_wheel">
+	<gazebo reference="caster_wheel_back">
+		<material>Gazebo/Black</material>
+		<mu1 value="0.001"/>
+		<mu2 value="0.001"/>
+	</gazebo>
+	<!-- CASTER WHEEL LINK 2 -->
+	<joint name="caster_wheel_joint_front" type="fixed">
+		<parent link="chassis"/>
+		<child link="caster_wheel_front"/>
+		<origin xyz="0.1 0 0"/>
+	</joint>
+	<link name="caster_wheel_front">
+		<visual>
+			<geometry>
+				<sphere radius="0.04"/>
+			</geometry>
+			<material name="black"/>
+		</visual>
+		<collision>
+			<geometry>
+				<sphere radius="0.04"/>
+			</geometry>
+			<material name="black"/>
+		</collision>
+		<xacro:inertial_sphere mass="0.1" radius="0.04">
+			<origin xyz="0 0 0" rpy="0 0 0"/>
+		</xacro:inertial_sphere>
+	</link>
+	<gazebo reference="caster_wheel_front">
 		<material>Gazebo/Black</material>
 		<mu1 value="0.001"/>

File: description/ros2_control.xacro (robot description, xacro)
@@ -1,29 +1,62 @@
 <?xml version="1.0"?>
 <robot xmlns:xacro="http://www.ros.org/wiki/xacro">
-    <ros2_control name="GazeboSystem" type="system">
-    	<hardware>
-    		<plugin>gazebo_ros2_control/GazeboSystem</plugin>
-    	</hardware>
-    	<joint name="left_wheel_joint">
-    		<command_interface name="velocity">
-    			<param name="min">-10</param>
-    			<param name="max">10</param>
-    		</command_interface>
-    		<state_interface name="velocity"/>
-    		<state_interface name="position"/>
-    	</joint>
-    	<joint name="right_wheel_joint">
-    		<command_interface name="velocity">
-    			<param name="min">-10</param>
-    			<param name="max">10</param>
-    		</command_interface>
-    		<state_interface name="velocity"/>
-    		<state_interface name="position"/>
-    	</joint>
-	</ros2_control>
-	<gazebo>
-    	<plugin name="gazebo_ros2_control" filename="libgazebo_ros2_control.so">
-    		<parameters>$(find sim_bot)/config/my_controllers.yaml</parameters>
-    	</plugin>
-    </gazebo>
+    <xacro:unless value="$(arg sim_mode)">
+        <ros2_control name="RealRobot" type="system">
+            <hardware>
+                <plugin>diffdrive_arduino/DiffDriveArduinoHardware</plugin>
+                <param name="left_wheel_name">left_wheel_joint</param>
+                <param name="right_wheel_name">right_wheel_joint</param>
+                <param name="loop_rate">30</param>
+                <param name="device">/dev/ttyUSB0</param>
+                <param name="baud_rate">57600</param>
+                <param name="timeout_ms">1000</param>
+                <param name="enc_counts_per_rev">3436</param>
+            </hardware>
+            <joint name="left_wheel_joint">
+                <command_interface name="velocity">
+                    <param name="min">-10</param>
+                    <param name="max">10</param>
+                </command_interface>
+                <state_interface name="position"/>
+                <state_interface name="velocity"/>
+            </joint>
+            <joint name="right_wheel_joint">
+                <command_interface name="velocity">
+                    <param name="min">-10</param>
+                    <param name="max">10</param>
+                </command_interface>
+                <state_interface name="position"/>
+                <state_interface name="velocity"/>
+            </joint>
+        </ros2_control>
+    </xacro:unless>
+    <xacro:if value="$(arg sim_mode)">
+        <ros2_control name="GazeboSystem" type="system">
+            <hardware>
+			    <plugin>gz_ros2_control/GazeboSimSystem</plugin>
+			</hardware>
+			<joint name="left_wheel_joint">
+                <command_interface name="velocity">
+                    <param name="min">-10</param>
+                    <param name="max">10</param>
+                </command_interface>
+                <state_interface name="velocity"/>
+                <state_interface name="position"/>
+            </joint>
+            <joint name="right_wheel_joint">
+                <command_interface name="velocity">
+                    <param name="min">-10</param>
+                    <param name="max">10</param>
+                </command_interface>
+                <state_interface name="velocity"/>
+                <state_interface name="position"/>
+            </joint>
+        </ros2_control>
+    </xacro:if>
+    <gazebo>
+		<plugin name="gz_ros2_control::GazeboSimROS2ControlPlugin" filename="libgz_ros2_control-system.so">
+		    <parameters>$(find articubot_one)/config/my_controllers.yaml</parameters>
+            <parameters>$(find articubot_one)/config/gaz_ros2_ctl_use_sim.yaml</parameters>
+        </plugin>
+	</gazebo>
 </robot>
