Commit message: Update for ROS Jazzy and Gazebo Harmonic

File: description/tof_sensors.xacro (robot description, xacro)
@@ -2,784 +2,784 @@
 <robot xmlns:xacro="http://www.ros.org/wiki/xacro">
 	<!-- CENTRAL GROUP -->
-	<!-- S1 central ultrasonic  -->
-	<joint name="s1_ultrasonic_joint" type="fixed">
-		<parent link="chassis"/>
-		<child link="s1_ultrasonic_frame"/>
+	<!-- S0 central infrared  -->
+	<joint name="s0_infrared_joint" type="fixed">
+		<parent link="chassis"/>
+		<child link="s0_infrared_frame"/>
 		<origin xyz="0.14 0 0.09" rpy="0 0 0"/>
 	</joint>
-	<link name="s1_ultrasonic_frame">
-		<visual>
-			<geometry>
-				<box size="0.015 0.045 0.02"/>
-			</geometry>
-			<material name="red"/>
-		</visual>
-		<collision>
-			<geometry>
-				<box size="0.015 0.045 0.02"/>
-			</geometry>
-			<material name="red"/>
-		</collision>
-		<xacro:inertial_box mass="0.01" x="0.015" y="0.045" z="0.02">
-			<origin xyz="0 0 0" rpy="0 0 0"/>
-		</xacro:inertial_box>
-	</link>
-	<gazebo reference="s1_ultrasonic_frame">
-		<material>Gazebo/Red</material>
-        <sensor name="ultrasonic_s1" type="ray">
-            <pose> 0 0 0 0 0 0 </pose>
-            <visualize>true</visualize>
-            <update_rate>5</update_rate>
-            <ray>
-                <scan>
-                    <horizontal>
-                        <samples>30</samples>
-                        <resolution>1.000000</resolution>
-                        <min_angle>-0.12</min_angle>
-                        <max_angle>0.12</max_angle>
-                    </horizontal>
-                    <vertical>
-          				<samples>5</samples>
-          				<resolution>1.000000</resolution>
-          				<min_angle>-0.01</min_angle>
-          				<max_angle>0.01</max_angle>
-        			</vertical>
-                </scan>
-                <range>
-                    <min>0.02</min>
-                    <max>1.5</max>
-                    <resolution>0.01</resolution>
-                </range>
-                <noise>
-        			<type>gaussian</type>
-        			<mean>0.0</mean>
-        			<stddev>0.01</stddev>
-      			</noise>
-            </ray>
-            <plugin name="ultrasonic_s1" filename="libgazebo_ros_ray_sensor.so">
+	<link name="s0_infrared_frame">
+		<visual>
+			<geometry>
+				<box size="0.015 0.045 0.02"/>
+			</geometry>
+			<material name="red"/>
+		</visual>
+		<collision>
+			<geometry>
+				<box size="0.015 0.045 0.02"/>
+			</geometry>
+			<material name="red"/>
+		</collision>
+		<xacro:inertial_box mass="0.01" x="0.015" y="0.045" z="0.02">
+			<origin xyz="0 0 0" rpy="0 0 0"/>
+		</xacro:inertial_box>
+	</link>
+	<gazebo reference="s0_infrared_frame">
+		<material>Gazebo/Red</material>
+        <sensor name="infrared_s0" type="ray">
+            <pose> 0 0 0 0 0 0 </pose>
+            <visualize>true</visualize>
+            <update_rate>5</update_rate>
+            <ray>
+                <scan>
+                    <horizontal>
+                        <samples>30</samples>
+                        <resolution>1.000000</resolution>
+                        <min_angle>-0.05</min_angle>
+                        <max_angle>0.05</max_angle>
+                    </horizontal>
+                    <vertical>
+          				<samples>30</samples>
+          				<resolution>1.000000</resolution>
+          				<min_angle>-0.05</min_angle>
+                        <max_angle>0.05</max_angle>
+        			</vertical>
+                </scan>
+                <range>
+                    <min>0.02</min>
+                    <max>1.5</max>
+                    <resolution>0.01</resolution>
+                </range>
+                <noise>
+        			<type>gaussian</type>
+        			<mean>0.0</mean>
+        			<stddev>0.01</stddev>
+      			</noise>
+            </ray>
+            <plugin name="infrared_s0" filename="libgazebo_ros_ray_sensor.so">
+                <ros>
+                    <argument>~/out:=front_sonars/s0</argument>
+                </ros>
+                <output_type>sensor_msgs/Range</output_type>
+                <radiation_type>infrared</radiation_type>
+                <frame_name>s0_infrared_frame</frame_name>
+            </plugin>
+        </sensor>
+    </gazebo>
+    <!-- S1 left infrared-->
+	<joint name="s1_infrared_joint" type="fixed">
+		<parent link="chassis"/>
+		<child link="s1_infrared_frame"/>
+		<origin xyz="0.1275 0.04665 0.09" rpy="0 0 ${pi/6}"/>
+	</joint>
+	<link name="s1_infrared_frame">
+		<visual>
+			<geometry>
+				<box size="0.015 0.045 0.02"/>
+			</geometry>
+			<material name="red"/>
+		</visual>
+		<collision>
+			<geometry>
+				<box size="0.015 0.045 0.02"/>
+			</geometry>
+			<material name="red"/>
+		</collision>
+		<xacro:inertial_box mass="0.01" x="0.015" y="0.045" z="0.02">
+			<origin xyz="0 0 0" rpy="0 0 0"/>
+		</xacro:inertial_box>
+	</link>
+	<gazebo reference="s1_infrared_frame">
+		<material>Gazebo/Red</material>
+        <sensor name="infrared_s1" type="ray">
+            <pose> 0 0 0 0 0 0 </pose>
+            <visualize>true</visualize>
+            <update_rate>5</update_rate>
+            <ray>
+                <scan>
+                    <horizontal>
+                        <samples>30</samples>
+                        <resolution>1.000000</resolution>
+                        <min_angle>-0.05</min_angle>
+                        <max_angle>0.05</max_angle>
+                    </horizontal>
+                    <vertical>
+          				<samples>30</samples>
+          				<resolution>1.000000</resolution>
+          				<min_angle>-0.05</min_angle>
+                        <max_angle>0.05</max_angle>
+        			</vertical>
+                </scan>
+                <range>
+                    <min>0.02</min>
+                    <max>1.5</max>
+                    <resolution>0.01</resolution>
+                </range>
+                <noise>
+        			<type>gaussian</type>
+        			<mean>0.0</mean>
+        			<stddev>0.01</stddev>
+      			</noise>
+            </ray>
+            <plugin name="infrared_s1" filename="libgazebo_ros_ray_sensor.so">
                 <ros>
                     <argument>~/out:=front_sonars/s1</argument>
                 </ros>
                 <output_type>sensor_msgs/Range</output_type>
-                <radiation_type>ultrasound</radiation_type>
-                <frame_name>s1_ultrasonic_frame</frame_name>
-            </plugin>
-        </sensor>
-    </gazebo>
-    <!-- S12 left ultrasonic-->
-	<joint name="s12_ultrasonic_joint" type="fixed">
-		<parent link="chassis"/>
-		<child link="s12_ultrasonic_frame"/>
-		<origin xyz="0.1275 0.04665 0.09" rpy="0 0 ${pi/6}"/>
-	</joint>
-	<link name="s12_ultrasonic_frame">
-		<visual>
-			<geometry>
-				<box size="0.015 0.045 0.02"/>
-			</geometry>
-			<material name="red"/>
-		</visual>
-		<collision>
-			<geometry>
-				<box size="0.015 0.045 0.02"/>
-			</geometry>
-			<material name="red"/>
-		</collision>
-		<xacro:inertial_box mass="0.01" x="0.015" y="0.045" z="0.02">
-			<origin xyz="0 0 0" rpy="0 0 0"/>
-		</xacro:inertial_box>
-	</link>
-	<gazebo reference="s12_ultrasonic_frame">
-		<material>Gazebo/Red</material>
-        <sensor name="ultrasonic_s12" type="ray">
-            <pose> 0 0 0 0 0 0 </pose>
-            <visualize>true</visualize>
-            <update_rate>5</update_rate>
-            <ray>
-                <scan>
-                    <horizontal>
-                        <samples>30</samples>
-                        <resolution>1.000000</resolution>
-                        <min_angle>-0.12</min_angle>
-                        <max_angle>0.12</max_angle>
-                    </horizontal>
-                    <vertical>
-          				<samples>5</samples>
-          				<resolution>1.000000</resolution>
-          				<min_angle>-0.01</min_angle>
-          				<max_angle>0.01</max_angle>
-        			</vertical>
-                </scan>
-                <range>
-                    <min>0.02</min>
-                    <max>1.5</max>
-                    <resolution>0.01</resolution>
-                </range>
-                <noise>
-        			<type>gaussian</type>
-        			<mean>0.0</mean>
-        			<stddev>0.01</stddev>
-      			</noise>
-            </ray>
-            <plugin name="ultrasonic_s12" filename="libgazebo_ros_ray_sensor.so">
-                <ros>
-                    <argument>~/out:=front_sonars/s12</argument>
-                </ros>
-                <output_type>sensor_msgs/Range</output_type>
-                <radiation_type>ultrasound</radiation_type>
-                <frame_name>s12_ultrasonic_frame</frame_name>
-            </plugin>
-        </sensor>
-    </gazebo>
-    <!-- S2 right ultrasonic -->
-	<joint name="s2_ultrasonic_joint" type="fixed">
-		<parent link="chassis"/>
-		<child link="s2_ultrasonic_frame"/>
+                <radiation_type>infrared</radiation_type>
+                <frame_name>s1_infrared_frame</frame_name>
+            </plugin>
+        </sensor>
+    </gazebo>
+    <!-- S11 right infrared -->
+	<joint name="s11_infrared_joint" type="fixed">
+		<parent link="chassis"/>
+		<child link="s11_infrared_frame"/>
 		<origin xyz="0.1275 -0.04665 0.09" rpy="0 0 -${pi/6}"/>
 	</joint>
-	<link name="s2_ultrasonic_frame">
-		<visual>
-			<geometry>
-				<box size="0.015 0.045 0.02"/>
-			</geometry>
-			<material name="red"/>
-		</visual>
-		<collision>
-			<geometry>
-				<box size="0.015 0.045 0.02"/>
-			</geometry>
-			<material name="red"/>
-		</collision>
-		<xacro:inertial_box mass="0.01" x="0.015" y="0.045" z="0.02">
-			<origin xyz="0 0 0" rpy="0 0 0"/>
-		</xacro:inertial_box>
-	</link>
-	<gazebo reference="s2_ultrasonic_frame">
-		<material>Gazebo/Red</material>
-        <sensor name="ultrasonic_s2" type="ray">
-            <pose> 0 0 0 0 0 0 </pose>
-            <visualize>true</visualize>
-            <update_rate>5</update_rate>
-            <ray>
-                <scan>
-                    <horizontal>
-                        <samples>30</samples>
-                        <resolution>1.000000</resolution>
-                        <min_angle>-0.12</min_angle>
-                        <max_angle>0.12</max_angle>
-                    </horizontal>
-                    <vertical>
-          				<samples>5</samples>
-          				<resolution>1.000000</resolution>
-          				<min_angle>-0.01</min_angle>
-          				<max_angle>0.01</max_angle>
-        			</vertical>
-                </scan>
-                <range>
-                    <min>0.02</min>
-                    <max>1.5</max>
-                    <resolution>0.01</resolution>
-                </range>
-                <noise>
-        			<type>gaussian</type>
-        			<mean>0.0</mean>
-        			<stddev>0.01</stddev>
-      			</noise>
-            </ray>
-            <plugin name="ultrasonic_s2" filename="libgazebo_ros_ray_sensor.so">
-                <ros>
-                    <argument>~/out:=front_sonars/s2</argument>
-                </ros>
-                <output_type>sensor_msgs/Range</output_type>
-                <radiation_type>ultrasound</radiation_type>
-                <frame_name>s2_ultrasonic_frame</frame_name>
+	<link name="s11_infrared_frame">
+		<visual>
+			<geometry>
+				<box size="0.015 0.045 0.02"/>
+			</geometry>
+			<material name="red"/>
+		</visual>
+		<collision>
+			<geometry>
+				<box size="0.015 0.045 0.02"/>
+			</geometry>
+			<material name="red"/>
+		</collision>
+		<xacro:inertial_box mass="0.01" x="0.015" y="0.045" z="0.02">
+			<origin xyz="0 0 0" rpy="0 0 0"/>
+		</xacro:inertial_box>
+	</link>
+	<gazebo reference="s11_infrared_frame">
+		<material>Gazebo/Red</material>
+        <sensor name="infrared_s11" type="ray">
+            <pose> 0 0 0 0 0 0 </pose>
+            <visualize>true</visualize>
+            <update_rate>5</update_rate>
+            <ray>
+                <scan>
+                    <horizontal>
+                        <samples>30</samples>
+                        <resolution>1.000000</resolution>
+                        <min_angle>-0.05</min_angle>
+                        <max_angle>0.05</max_angle>
+                    </horizontal>
+                    <vertical>
+          				<samples>30</samples>
+          				<resolution>1.000000</resolution>
+          				<min_angle>-0.05</min_angle>
+                        <max_angle>0.05</max_angle>
+        			</vertical>
+                </scan>
+                <range>
+                    <min>0.02</min>
+                    <max>1.5</max>
+                    <resolution>0.01</resolution>
+                </range>
+                <noise>
+        			<type>gaussian</type>
+        			<mean>0.0</mean>
+        			<stddev>0.01</stddev>
+      			</noise>
+            </ray>
+            <plugin name="infrared_s11" filename="libgazebo_ros_ray_sensor.so">
+                <ros>
+                    <argument>~/out:=front_sonars/s11</argument>
+                </ros>
+                <output_type>sensor_msgs/Range</output_type>
+                <radiation_type>infrared</radiation_type>
+                <frame_name>s11_infrared_frame</frame_name>
             </plugin>
         </sensor>
     </gazebo>
     <!-- RIGHT GROUP -->
-	<!-- S4 central ultrasonic  -->
-	<joint name="s4_ultrasonic_joint" type="fixed">
-		<parent link="chassis"/>
-		<child link="s4_ultrasonic_frame"/>
+	<!-- S9 central infrared  -->
+	<joint name="s9_infrared_joint" type="fixed">
+		<parent link="chassis"/>
+		<child link="s9_infrared_frame"/>
 		<origin xyz="0 -0.13 0.09" rpy="0 0 -${pi/2}"/>
 	</joint>
-	<link name="s4_ultrasonic_frame">
-		<visual>
-			<geometry>
-				<box size="0.015 0.045 0.02"/>
-			</geometry>
-			<material name="red"/>
-		</visual>
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